File: AD9744 Ersatz Eval Board Rev. A.kicad_pcb (KiCad board)
At the start: 2 copper layers, 48 x 48 mm, 42 parts, among them J1 Conn_02x09, J2 SMA, J3 SMA, J4 Screw Terminal 01x02, U1 AD97444ARUZRL7

Commit message: Release A1
Parts:
- R2, R6: value 50 -> 62
- R5: value 2k -> 2.37k
- TR1: value T1-6T+ -> T2-1T+
Changed lines of the file:
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@@
 			)
 		)
-		(property "Value" "50"
+		(property "Value" "62"
 			(at 0 1.43 90)
 			(layer "F.Fab")
@@
 			)
 		)
-		(property "Value" "50"
+		(property "Value" "62"
 			(at 0 1.43 90)
 			(layer "F.Fab")
@@
 		(sheetname "Root")
 		(sheetfile "AD9744 Ersatz Eval Board Rev. A.kicad_sch")
-		(attr smd dnp)
+		(attr smd)
 		(fp_line
 			(start -0.146267 0.51)
@@
 		(sheetname "Root")
 		(sheetfile "AD9744 Ersatz Eval Board Rev. A.kicad_sch")
-		(attr smd dnp)
+		(attr smd)
 		(fp_line
 			(start -0.254724 0.5225)
@@
 			)
 		)
-		(property "Value" "2k"
+		(property "Value" "2.37k"
 			(at 0 1.43 0)
 			(layer "F.Fab")
@@
 			)
 		)
-		(property "Description" "1%"
+		(property "Description" "0.5%"
 			(at 0 0 0)
 			(unlocked yes)
@@
 			)
 		)
+		(property "Temp Stability" "25 PPM/C"
+			(at 0 0 0)
+			(unlocked yes)
+			(layer "F.Fab")
+			(hide yes)
+			(effects
+				(font
+					(size 1 1)
+					(thickness 0.15)
+				)
+			)
+		)
 		(property ki_fp_filters "R_*")
 		(sheetname "Root")
@@
 		(sheetname "Root")
 		(sheetfile "AD9744 Ersatz Eval Board Rev. A.kicad_sch")
-		(attr smd dnp)
+		(attr smd)
 		(fp_line
 			(start -0.146267 -0.51)
@@
 			)
 		)
-		(property "Description" "16V, X5R"
+		(property "Description" "16V, X7R"
 			(at 0 0 -90)
 			(unlocked yes)
@@
 		(sheetname "Root")
 		(sheetfile "AD9744 Ersatz Eval Board Rev. A.kicad_sch")
-		(attr smd dnp)
+		(attr smd)
 		(fp_line
 			(start -0.254724 0.5225)
@@
 			)
 		)
-		(property "Description" "16V, X5R"
+		(property "Description" "16V, X7R"
 			(at 0 0 -90)
 			(unlocked yes)
@@
 			)
 		)
-		(property "Value" "T1-6T+"
+		(property "Value" "T2-1T+"
 			(at 3.81 7.41 0)
 			(layer "F.Fab")
